File: Grove expansion v5.sch (EAGLE design)
At the start: 57 parts, among them J1 16p-2.54, J2 16p-2.54, P1A TP0602N3, P1B SSM3J328R,LF, P2A TP0602N3, P2B SSM3J328R,LF, P3A TP0602N3, P3B SSM3J328R,LF

Commit message: Add files via upload
Parts:
- removed J1, J2: 16p-2.54, OPL_Connector:DIP-BLACK-MALE-HEADER-VERT(16P-2.54)
- added CN1, CN2, CN3, CN4: 8p-2.54, OPL_Connector:DIP-BLACK-FEMALE-HEADER-VERT(8P-2.54)
Connections:
- net +3V3: now also CN3.3; no longer J2.3
- net +5V: now also CN3.1; no longer J2.1
- net BUTTON: now also CN4.5; no longer J2.13
- net GND: now also CN3.2; no longer J2.2
- net GPS_RX: now also CN3.5; no longer J2.5
- net GPS_TX: now also CN3.6; no longer J2.6
- net LOPY_CLK: now also CN1.7; no longer J1.7
- net LOPY_MISO: now also CN2.1; no longer J1.9
- net LOPY_MOSI: now also CN1.8; no longer J1.8
- net P13: now also CN4.6; no longer J2.14
- net P15: now also CN4.4; no longer J2.12
- net P16: now also CN4.3; no longer J2.11
- net PM1_RX: now also CN4.2; no longer J2.10
- net PM1_TX: now also CN1.5; no longer J1.5
- net PM2_RX: now also CN4.1; no longer J2.9
- net PM2_TX: now also CN2.5; no longer J1.13
- net RGB_LED: now also CN1.4; no longer J1.4
- net RST: now also CN1.1; no longer J1.1
- net RX0: now also CN1.2; no longer J1.2
- net RXD1: now also CN1.6; no longer J1.6
- net SCL: now also CN2.4; no longer J1.12
- net SDA: now also CN2.3; no longer J1.11
- net SD_CLK: now also CN3.4; no longer J2.4
- net SD_DO: now also CN2.2; no longer J1.10
- net TR1_C: now also CN3.7; no longer J2.7
- net TR3_C: now also CN3.8; no longer J2.8
- net TX0: now also CN1.3; no longer J1.3
- net WIFI: now also CN2.6; no longer J1.14
